File: Power.kicad_sch (KiCad schematic)
At the start: 0 parts

Commit message: Finished power and phase blocks
Parts:
- added C35, C36, C8: T521D107M025ATE040, easyeda2kicad:CAP-SMD_L7.3-W4.3, symbol easyeda_symbole:T521D107M025ATE040
- added C5, C6, C7: CL21A226MAYNNNE, easyeda2kicad:C0805, symbol easyeda_symbole:CL21A226MAYNNNE
- added CN1: XT60PW-M, easyeda2kicad:CONN-TH_XT60PW-M, symbol easyeda2kicad:XT60PW-M
- added D2: B540C-13-F, easyeda2kicad:SMC_L7.1-W6.2-LS8.1-RD, symbol easyeda_symbole:B540C-13-F
- added D6, D7: 0603ESDA-05N, easyeda2kicad:D0603-BI, symbol easyeda2kicad:0603ESDA-05N
- added H1, H2, H3, H4: MountingHole_Pad, MountingHole:MountingHole_2.2mm_M2_Pad, symbol Mechanical:MountingHole_Pad
- added LED1: KT-0603G, easyeda2kicad:LED0603-RD, symbol easyeda_symbole:0603Green509-620mcd
- added R14, R15: 0603WAF5101T5E, easyeda2kicad:R0603, symbol easyeda2kicad:0603WAF5101T5E
- added R18: 0603WAF1000T5E, easyeda2kicad:R0603, symbol easyeda_symbole:0603WAF1000T5E
- added U7: TPSPX3819M5-L-3-3, easyeda2kicad:SOT-23-5_L3.0-W1.6-P0.95-LS2.8-BR, symbol easyeda_symbole:TPSPX3819M5-L-3-3
- added USB1: TYPE-C 6P(073), easyeda2kicad:TYPE-C-SMD_TYPE-C-6P_5, symbol easyeda_symbole:TYPE-C6P(073)
Connections:
- new net: LED1.2 (A), R18.1
- new net +3.3V: C6.2, R18.2, U7.5 (VOUT)
- new net +VBAT: C35.1, C36.1, C5.2, C7.2, C8.1, CN1.2 (+), D2.1 (K), U7.1 (VIN), U7.3 (EN)
- new net CC1: R14.2, USB1.A5 (CC1)
- new net CC2: R15.2, USB1.B5 (CC2)
- new net GND: C35.2, C36.2, C5.1, C6.1, C7.1, C8.2, CN1.1 (-), CN1.3, CN1.4, D6.1, D7.1, H1.1, H2.1, H3.1, H4.1, LED1.1 (K), R14.1, R15.1, U7.2 (GND), USB1.7 (EH), USB1.A12 (GND), USB1.B12 (GND)
- new net USB_5V: D2.2 (A), D6.2, D7.2, USB1.A9 (VBUS), USB1.B9 (VBUS)
Other:
- note added: "5V OR 4S(16.8V) TO 3.3V"
- note added: "when both 4s and usb connected to prevent reach usb"
