File: stm32.kicad_sch (KiCad schematic)
At the start: 64 parts, among them CN2 XY308-2.54-4P, CN3 SM04B-SRSS-TB (LF)(SN), CN4 SM04B-SRSS-TB (LF)(SN), SW2 6.0*6.0*6.0, SW3 6.0*6.0*6.0, U1 STM32G431CBT6, U2 DRV8323SRTAR, U3 TMC2209-LA-T, U4 DRV8876PWPR, U5 ABM8-272-T3_C20625731, U6 HB-PH9-12727PB2GOB, U8 XY308-2.54-2P

Commit message: some improvments - new pinout is ok
Parts:
- removed R30: 0603WAF1002T5E, easyeda2kicad:R0603, symbol easyeda2kicad:0603WAF1002T5E
- removed R34, R37, R40: 0603WAF4701T5E, easyeda2kicad:R0603, symbol easyeda2kicad:0603WAF4701T5E
- added C58, C61, C62: CC0603KRX7R9BB104, easyeda2kicad:C0603, symbol easyeda2kicad:CC0603KRX7R9BB104
- added R29, R31, R38: 0603WAF1000T5E, easyeda2kicad:R0603, symbol easyeda2kicad:0603WAF1000T5E
Connections:
- net GND: now also C58.2, C61.2, C62.2
- net I2C1_SCL_R: now reaches R28.1
- net I2C1_SCL_R: now also U1.39 (PA15)
- net I2C3_SCL renamed I2C1_SCL
- net I2C1_SCL: no longer U1.39 (PA15)
- net I2C3_SDA renamed I2C1_SDA
- net UART_PDN_RX renamed STM32_UART1_RX
- net STM32_UART1_RX: now also U1.44 (PB7); no longer U1.43 (PB6)
- net UART_PDN_TX renamed STM32_UART1_TX
- net STM32_UART1_TX: now also U1.43 (PB6); no longer U1.44 (PB7)
- net VSENSE_A renamed BLDC_VSENSE_A
- net BLDC_VSENSE_A: now also C62.1, R31.2
- net VSENSE_B renamed BLDC_VSENSE_B
- net BLDC_VSENSE_B: now also C61.1, R38.2
- net VSENSE_C renamed BLDC_VSENSE_C
- net BLDC_VSENSE_C: now also C58.1, R29.1
- new net VSENSE_PHASE_A: R31.1
- new net VSENSE_PHASE_B: R38.1
- new net VSENSE_PHASE_C: R29.2
- no-connect marks 12 -> 14
Other:
- note added: "NRST has an internal pullup"
- moved on the sheet: R28
